File: KiCAD_files/Measurment.sch (KiCad schematic (older format))
At the start: 38 parts, among them J1 Board_outline, U1 NMA1505SC, U2 AMC1100, U3 AMC1100, U4 AMC1311, U5 NMA1505SC

Commit message: Major modifications of the measurment board schematic Component placement finalized - 3D footprints added - mezzanine assembly on freecad added
Parts:
- removed J1: Board_outline, Footprints:Board outline, symbol Symbols:Board_outline
- removed U5: NMA1505SC, Converter_DCDC:Converter_DCDC_muRata_NMAxxxxSC_THT, symbol Regulator_Switching:NMA1505SC
- added C10, C11, C12, C13, C14, C15, C16, C7, C8, C9: C_Small, Capacitor_SMD:C_0805_2012Metric, symbol Device:C_Small
- added D1: D_TVS, Diode_SMD:D_SMB, symbol Device:D_TVS
- added D2, D3, D4, D5, D6: LED, LED_SMD:LED_0805_2012Metric, symbol Device:LED
- added J1: Measurment_stage_outline_outputs, Footprints:Measurment_stage_outline_outputs, symbol Symbols:Measurment_stage_outline_outputs
- added J2: Measurment_stage_outline_signal_inputs, Footprints:Measurment_stage_outline_inputs, symbol Symbols:Measurment_stage_outline_signal_inputs
- added J3: Conn_01x02, Connector_Phoenix_MC:PhoenixContact_MC_1,5_2-G-3.81_1x02_P3.81mm_Horizontal, symbol Connector_Generic:Conn_01x02
- added R27, R28, R29, R30, R31, R32, R33, R34, R35, R36, R37: R_Small, Resistor_SMD:R_0805_2012Metric, symbol Device:R_Small
- added U5: R-78C5.0-1.0, Converter_DCDC:Converter_DCDC_RECOM_R-78E-0.5_THT, symbol Regulator_Switching:R-78C5.0-1.0
- added U6: AMS1117-3.3, Package_TO_SOT_SMD:SOT-223-3_TabPin2, symbol Regulator_Linear:AMS1117-3.3
- added U7: NMA1505SC, Converter_DCDC:Converter_DCDC_muRata_NMAxxxxSC_THT, symbol Regulator_Switching:NMA1505SC
- C1, C2, C3, C4, C5, C6: renamed from C?; footprint (none) -> Capacitor_SMD:C_0805_2012Metric
- gave numbers to parts that had none: 11
Connections:
- net labels added: VIHigh+_ADC, VIHigh-_ADC, VILow1+_ADC, VILow1-_ADC, VILow2+_ADC, VILow2_ADC
- wire segments 133 -> 240
Other:
- moved on the sheet: C1, C2, C3, C4, C5, C6, R1, R10, R11, R12, R13, R14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
