File: KiCAD_files/Microcontroller.kicad_sch (KiCad schematic)
At the start: 60 parts, among them J403 RJE721881411, J404 RJE721881411, P401 Power2, U401 OwnTech_SPIN, U402 TCAN334GDR, U405 LTC2850xS8, U406 MCP6487T-E/SN

Commit message: wip SHEMATIC
Parts:
- removed P401: Power2, symbol Symbols:Power2
- U401: DNP x -> (none); Functional Block Microcontroller -> (none)
Connections:
- net HRTIM_CHA1 renamed HRTIM_CHA1_DGND
- net HRTIM_CHA2 renamed HRTIM_CHA2_DGND
- net HRTIM_CHC1 renamed HRTIM_CHC1_DGND
- net HRTIM_CHC2 renamed HRTIM_CHC2_DGND
- net I_{I1Low} renamed I_{I1Low_DGND}
- net I_{I2Low} renamed I_{I2Low_DGND}
- net I_{IHigh} renamed I_{IHigh_sense_DGND}
- net V_{I1Low} renamed V_{I1Low_DGND}
- net V_{I2Low} renamed V_{I2Low_DGND}
- net V_{IHigh} renamed V_{IHigh_sense_DGND}
- net ~{STBY1} renamed ~{STBY1}_DGND
- net ~{STBY2} renamed ~{STBY2}_DGND
Other:
- note added: "Simulation available https://tinyurl.com/2qg7lcok"
- note removed: "Simulation available"
- note removed: "https://tinyurl.com/2qg7lcok"
- company: https://gitlab.laas.fr/owntech/1leg/-/tree/V1.1.2/KiCAD_files -> https://gitlab.laas.fr/owntech/boards/TWIST
- moved on the sheet: C401, JP401, JP404, JP412, JP413, R401, U402

Commit message: big clean in libraries (imported components in symbol), PCB WIP
Parts:
- D403: symbol Diode:1N4148WS -> Symbols:PMEG2010AEJ,115; Functional Block Communication -> Driver; Subfunction Analog bus -> Gate circuit
- TH401, TH402: footprint Connector_PinHeader_1.27mm:PinHeader_1x02_P1.27mm_Vertical -> Connector_PinHeader_2.54mm:PinHeader_1x02_P2.54mm_Vertical
Changed lines of the file:
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@@
     (effects (font (size 1.27 1.27)) (justify left))
+  )
+  (hierarchical_label "LEG1_CAPA_DRIVE_DGND" (shape output) (at 283.21 45.72 180) (fields_autoplaced)
+    (effects (font (size 1.27 1.27)) (justify right))
   )
   (hierarchical_label "~{STBY1}_DGND" (shape output) (at 144.78 27.94 0) (fields_autoplaced)
@@
   (hierarchical_label "~{STBY2}_DGND" (shape output) (at 144.78 21.59 0) (fields_autoplaced)
     (effects (font (size 1.27 1.27)) (justify left))
+  )
+  (hierarchical_label "LEG2_CAPA_DRIVE_DGND" (shape output) (at 283.21 50.8 180) (fields_autoplaced)
+    (effects (font (size 1.27 1.27)) (justify right))
   )
   (hierarchical_label "I_{I2Low_DGND}" (shape input) (at 93.98 72.39 0) (fields_autoplaced)
@@
       (effects (font (size 1.27 1.27)) (justify left))
     )
-    (property "Footprint" "Connector_PinHeader_1.27mm:PinHeader_1x02_P1.27mm_Vertical" (at 168.91 105.41 0)
+    (property "Footprint" "Connector_PinHeader_2.54mm:PinHeader_1x02_P2.54mm_Vertical" (at 168.91 105.41 0)
       (effects (font (size 1.27 1.27)) hide)
     )
@@
     )
   )
-  (symbol (lib_id "Symbols:OwnTech_SPIN") (at 60.96 30.48 0) (unit 1)
+  (symbol (lib_name "OwnTech_SPIN_1") (lib_id "Symbols:OwnTech_SPIN") (at 60.96 30.48 0) (unit 1)
     (in_bom yes) (on_board yes) (dnp no) (fields_autoplaced)
     (property "Reference" "U401" (at 73.66 24.13 0)
@@
     )
   )
-  (symbol (lib_id "Diode:1N4148WS") (at 90.17 161.29 0) (mirror y) (unit 1)
+  (symbol (lib_id "Symbols:PMEG2010AEJ,115") (at 90.17 161.29 0) (mirror y) (unit 1)
     (in_bom yes) (on_board yes) (dnp no)
     (property "Reference" "D403" (at 90.17 163.83 0)
@@
       (effects (font (size 1.27 1.27)))
     )
-    (property "Footprint" "Diode_SMD:D_SOD-323_HandSoldering" (at 90.17 165.735 0)
-      (effects (font (size 1.27 1.27)) hide)
-    )
-    (property "Datasheet" "https://www.vishay.com/docs/85751/1n4148ws.pdf" (at 90.17 161.29 0)
+    (property "Footprint" "Diode_SMD:D_SOD-323_HandSoldering" (at 90.17 161.29 0)
+      (effects (font (size 1.27 1.27)) hide)
+    )
+    (property "Datasheet" "~" (at 90.17 161.29 0)
       (effects (font (size 1.27 1.27)) hide)
     )
@@
       (effects (font (size 1.27 1.27)) hide)
     )
-    (property "Functional Block" "Communication" (at 90.17 161.29 0)
+    (property "Functional Block" "Driver" (at 90.17 161.29 0)
       (effects (font (size 1.27 1.27)) hide)
     )
@@
       (effects (font (size 1.27 1.27)) hide)
     )
-    (property "Subfunction" "Analog bus" (at 90.17 161.29 0)
+    (property "Subfunction" "Gate circuit" (at 90.17 161.29 0)
       (effects (font (size 1.27 1.27)) hide)
     )
@@
       (effects (font (size 1.27 1.27)) (justify left))
     )
-    (property "Footprint" "Connector_PinHeader_1.27mm:PinHeader_1x02_P1.27mm_Vertical" (at 194.31 104.14 0)
-      (effects (font (size 1.27 1.27)) hide)
-    )
+    (property "Footprint" "Connector_PinHeader_2.54mm:PinHeader_1x02_P2.54mm_Vertical" (at 194.31 104.14 0)
+      (effects (font (size 1.27 1.27)) hide)
+    )

Commit message: Ready for design review
Parts:
- removed JP404: Jumper_2_Bridged, Jumper:SolderJumper-2_P1.3mm_Bridged_RoundedPad1.0x1.5mm, symbol Jumper:SolderJumper_2_Bridged
- TH401, TH402: footprint Connector_PinHeader_2.54mm:PinHeader_1x02_P2.54mm_Vertical -> Connector_PinHeader_2.00mm:PinHeader_1x02_P2.00mm_Vertical
Connections:
- net PC6 is gone; now on net LEG1_CAPA_DRIVE_DGND: U401.7 (PC6)
- net LEG2_CAPA_DRIVE_DGND: now also U401.56 (PB7)
- net HRTIM1_SCIN renamed HRTIM_SYNC
- net PB1 renamed PB1_HRTIM_SCOUT
- net PB6 renamed PB6_HRTIM_SCIN
- no-connect marks 25 -> 24
Other:
- moved on the sheet: C402, JP405, JP406, JP412, JP413, JP414, JP415, R406, R407, TH401, TH402, TP401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

Commit message: dev
Parts:
- TH401, TH402: value NXFT15XH103FA2B100 -> NXFT15XH103FA2B100
- U401: manf# (none) -> SPIN
Changed lines of the file:
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@@
       (effects (font (size 1.27 1.27)) (justify left))
     )
-    (property "Value" "NXFT15XH103FA2B100 " (at 211.455 112.395 0)
+    (property "Value" "NXFT15XH103FA2B100" (at 211.455 112.395 0)
       (effects (font (size 1.27 1.27)) (justify left))
     )
@@
     )
     (property "Datasheet" "" (at 68.58 30.48 0)
+      (effects (font (size 1.27 1.27)) hide)
+    )
+    (property "manf#" "SPIN" (at 69.85 30.48 0)
       (effects (font (size 1.27 1.27)) hide)
     )
@@
       (effects (font (size 1.27 1.27)) hide)
     )
+    (property "manf#" "SPIN" (at 55.88 91.44 0)
+      (effects (font (size 1.27 1.27)) hide)
+    )
     (pin "1")
     (pin "10")
@@
       (effects (font (size 1.27 1.27)) (justify left))
     )
-    (property "Value" "NXFT15XH103FA2B100 " (at 210.82 105.41 0)
+    (property "Value" "NXFT15XH103FA2B100" (at 210.82 105.41 0)
       (effects (font (size 1.27 1.27)) (justify left))
     )
@@
     )
     (property "Datasheet" "" (at 129.54 93.98 0)
+      (effects (font (size 1.27 1.27)) hide)
+    )
+    (property "manf#" "SPIN" (at 128.27 93.98 0)
       (effects (font (size 1.27 1.27)) hide)
     )
@@
       (effects (font (size 1.27 1.27)) hide)
     )
+    (property "manf#" "SPIN" (at 57.15 113.03 0)
+      (effects (font (size 1.27 1.27)) hide)
+    )

Commit message: ready for design review
Other:
- note added: "Analog share"
Changed lines of the file:
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@@
     (fill (type none))
   )
-  (text "CAN bus" (at 29.21 280.67 0)
-    (effects (font (size 2.54 2.54)) (justify left bottom))
-  )
-  (text "Communication RJ45 terminals " (at 120.65 280.67 0)
-    (effects (font (size 2.54 2.54)) (justify left bottom))
+  (text "CAN bus" (at 60.96 198.12 0)
+    (effects (font (size 2.54 2.54) (thickness 0.508) bold) (justify left bottom))
+  )
+  (text "Communication RJ45 terminals " (at 167.64 196.85 0)
+    (effects (font (size 2.54 2.54) (thickness 0.508) bold) (justify left bottom))
   )
   (text "Low pass filter\nResistor = 120R\nCap = 10nF\nCutoff freq = 132 kHz"
@@
     (effects (font (face "Arial") (size 1.27 1.27)) (justify left bottom))
   )
-  (text "SPIN Pinout" (at 30.48 20.32 0)
-    (effects (font (size 2.4892 2.4892)) (justify left bottom))
+  (text "SPIN Pinout" (at 73.66 19.05 0)
+    (effects (font (size 2.4892 2.4892) (thickness 0.4978) bold) (justify left bottom))
   )
   (text "Max current flowing: 0.16mA@125°C\nR0 = 10kOhm @T0 = 25°C\nB = 3450\nR = R0 * exp[B(T0-T)/T0*T]\nTemp expressed in °K"
@@
     (effects (font (size 1.27 1.27) (thickness 0.254) bold) (justify left bottom))
   )
-  (text "Emitting circuit" (at 27.94 189.23 0)
+  (text "Emitting circuit" (at 30.48 182.88 0)
     (effects (font (size 2.4892 2.4892)) (justify left bottom))
   )
   (text "Current sharing analog bus. Highest voltage is imposing its voltage to the bus"
-    (at 77.47 189.23 0)
+    (at 77.47 187.96 0)
     (effects (font (size 2 2)) (justify left bottom))
   )
@@
     (effects (font (size 2.4892 2.4892)) (justify left bottom))
   )
-  (text "RS485 Bus" (at 204.47 189.23 0)
-    (effects (font (size 2.54 2.54)) (justify left bottom))
-  )
-  (text "Receiving circuit" (at 138.43 180.34 0)
+  (text "RS485 Bus" (at 207.01 127 0)
+    (effects (font (size 2.54 2.54) (thickness 0.508) bold) (justify left bottom))
+  )
+  (text "Receiving circuit" (at 158.75 182.88 0)
     (effects (font (size 2.4892 2.4892)) (justify left bottom))
   )
   (text "Simulation available \nhttps://tinyurl.com/2qg7lcok"
-    (at 171.45 185.42 0)
+    (at 171.45 125.73 0)
     (effects (font (size 1.27 1.27)) (justify left bottom))
   )
@@
     (effects (font (size 1.27 1.27)) (justify left bottom))
   )
+  (text "Analog share" (at 101.6 125.73 0)
+    (effects (font (size 2.4892 2.4892) (thickness 0.4978) bold) (justify left bottom))
+  )
   (text "FALSTAD\nhttps://tinyurl.com/2262hpg6" (at 204.47 82.55 0)
     (effects (font (size 1.27 1.27)) (justify left bottom))
   )
   (text "Communication link encompasses \n- Analog bus \n- CAN bus \n- HRTIM sync\n- RS485 20Mbps bus"
-    (at 247.65 280.67 0)
+    (at 119.38 280.67 0)
     (effects (font (size 1.27 1.27)) (justify left bottom))
   )
@@
     )
   )
-  (symbol (lib_id "Symbols:OwnTech_SPIN") (at 55.88 91.44 0) (unit 2)
+  (symbol (lib_name "OwnTech_SPIN_2") (lib_id "Symbols:OwnTech_SPIN") (at 55.88 91.44 0) (unit 2)
     (in_bom yes) (on_board yes) (dnp no)
     (property "Reference" "U401" (at 59.69 90.17 0)
