File: KiCAD_files/High_side.kicad_sch (KiCad schematic)
At the start: 27 parts, among them U204 MCP6486UT-E/LT, U601 AMC1311DWV, U602 ACS723LLCTR-20AB-T

Commit message: acquisition chain resistor are now 0.5% tolerance
Parts:
- R217: manf# RT0805FRE075K9L -> RT0805DRE075K9L
- R? (x2): manf# RT0805FRE1320KL -> RT0805DRD0720KL
- R? (x4): manf# RT0805FRE1327KL -> RT0805DRD0727KL
Changed lines of the file:
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@@
       (effects (font (size 1.27 1.27)) hide)
     )
-    (property "manf#" "RT0805FRE1320KL" (at 226.06 180.34 0)
+    (property "manf#" "RT0805DRD0720KL" (at 226.06 180.34 0)
       (effects (font (size 1.27 1.27)) hide)
     )
@@
       (effects (font (size 1.27 1.27)) hide)
     )
-    (property "manf#" "RT0805FRE1327KL" (at 88.9 196.85 0)
+    (property "manf#" "RT0805DRD0727KL" (at 88.9 196.85 0)
       (effects (font (size 1.27 1.27)) hide)
     )
@@
       (effects (font (size 1.27 1.27)) hide)
     )
-    (property "manf#" "RT0805FRE075K9L" (at 240.03 208.28 0)
+    (property "manf#" "RT0805DRE075K9L" (at 240.03 208.28 0)
       (effects (font (size 1.27 1.27)) hide)
     )
@@
       (effects (font (size 1.27 1.27)) hide)
     )
-    (property "manf#" "RT0805FRE075K9L" (at 217.17 186.69 0)
+    (property "manf#" "RT0805DRE075K9L" (at 217.17 186.69 0)
       (effects (font (size 1.27 1.27)) hide)
     )
@@
       (effects (font (size 1.27 1.27)) hide)
     )
-    (property "manf#" "RT0805FRE1327KL" (at 116.84 210.82 0)
+    (property "manf#" "RT0805DRD0727KL" (at 116.84 210.82 0)
       (effects (font (size 1.27 1.27)) hide)
     )
@@
       (effects (font (size 1.27 1.27)) hide)
     )
-    (property "manf#" "RT0805FRE1327KL" (at 102.87 186.69 0)
+    (property "manf#" "RT0805DRD0727KL" (at 102.87 186.69 0)
       (effects (font (size 1.27 1.27)) hide)
     )
@@
       (effects (font (size 1.27 1.27)) hide)
     )
-    (property "manf#" "RT0805FRE1327KL" (at 88.9 191.77 0)
+    (property "manf#" "RT0805DRD0727KL" (at 88.9 191.77 0)
       (effects (font (size 1.27 1.27)) hide)
     )
@@
       (effects (font (size 1.27 1.27)) hide)
     )
-    (property "manf#" "RT0805FRE1320KL" (at 214.63 191.77 0)
-      (effects (font (size 1.27 1.27)) hide)
-    )
+    (property "manf#" "RT0805DRD0720KL" (at 214.63 191.77 0)
+      (effects (font (size 1.27 1.27)) hide)
+    )

Commit message: wip indus
Parts:
- C? (x2): footprint Footprints:C_0805_2012Metric -> Capacitor_SMD:C_1206_3216Metric; manf# C0805C104K5RACTU -> C1206C104K5RAC7867
Changed lines of the file:
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@@
   )
   (text "ACS712 is pin to pin compatible\nwith ACS723. If ACS712 is used,\nuntie pin 6 and place\nfilter capacitor on pin 6,\naccording to wanted BW.\n"
-    (at 144.78 35.56 0)
+    (at 143.51 35.56 0)
     (effects (font (size 1.27 1.27)) (justify left bottom))
   )
@@
       (effects (font (size 1.27 1.27)) (justify left))
     )
-    (property "Footprint" "Footprints:C_0805_2012Metric" (at 247.65 175.26 0)
+    (property "Footprint" "Capacitor_SMD:C_1206_3216Metric" (at 247.65 175.26 0)
       (effects (font (size 1.27 1.27)) hide)
     )
@@
       (effects (font (size 1.27 1.27)) hide)
     )
-    (property "manf#" "C0805C104K5RACTU" (at 247.65 175.26 0)
+    (property "manf#" "C1206C104K5RAC7867" (at 247.65 175.26 0)
       (effects (font (size 1.27 1.27)) hide)
     )
@@
       (effects (font (size 1.27 1.27)) (justify left))
     )
-    (property "Footprint" "Footprints:C_0805_2012Metric" (at 123.19 180.34 0)
+    (property "Footprint" "Capacitor_SMD:C_1206_3216Metric" (at 123.19 180.34 0)
       (effects (font (size 1.27 1.27)) hide)
     )
@@
       (effects (font (size 1.27 1.27)) hide)
     )
-    (property "manf#" "C0805C104K5RACTU" (at 123.19 180.34 0)
-      (effects (font (size 1.27 1.27)) hide)
-    )
+    (property "manf#" "C1206C104K5RAC7867" (at 123.19 180.34 0)
+      (effects (font (size 1.27 1.27)) hide)
+    )

Commit message: ready for design review
Parts:
- removed R?: 0R, Footprints:R_0805_2012Metric, symbol Device:R_Small
- removed U602: ACS723LLCTR-20AB-T, Package_SO:SOIC-8_3.9x4.9mm_P1.27mm, symbol Symbols:ACS723LLCTR-20AB-T
- added JP409: SolderJumper_2_Open, Jumper:SolderJumper-2_P1.3mm_Open_RoundedPad1.0x1.5mm, symbol Jumper:SolderJumper_2_Open
- added U602: +-20A Hall, Package_SO:SOIC-8_3.9x4.9mm_P1.27mm, symbol Symbols:ACS712ELCTR-20A-T
- C? (x2): Package 0805 -> 1206
- C?: DNP DNP -> (none)
Connections:
- net +5V_DGND: now also JP409.1 (A), U602.8 (VCC)
- net DGND: now also U602.5 (GND)
- net I_{IHighHall_DGND}: now also U602.7 (VIOUT)
- net V_{IHighOutFused_PGND}: now also U602.1 (IP+), U602.2 (IP+)
- net V_{IHigh_PGND}: now also U602.3 (IP-), U602.4 (IP-)
- net at C?.2: now also JP409.2 (B), U602.6 (FILTER)
Other:
- note added: "ACS712 direct equivalence: ACS724"
- note added: "ACS723 is pin to pin compatible with ACS712. If ACS723 is used, disconnect CA and tie pin 6 to either +5V or GND for wanted BW"
- note removed: "ACS712 is pin to pin compatible with ACS723. If ACS712 is used, untie pin 6 and place filter capacitor on pin 6, according to wanted BW."
